File: kicad/evereader/evereader.kicad_sch (KiCad schematic)
At the start: 56 parts, among them J1 USB_C_Receptacle_USB2.0_14P, J2 Micro_SD_Card_Det1, J3 Conn_02x04_Odd_Even, J4 Conn_02x04_Odd_Even, J5 Conn_01x02, J6 Conn_01x08, J7 Conn_01x08, J8 Conn_01x02, J9 Conn_01x02, Q1 FS8205A, SW1 SW_Push, SW2 SW_Push, SW3 SW_Push, SW4 SW_Push, SW5 SW_Push, U1 TP4056-42-ESOP8, U2 DW01A, U3 AP2112K-3.3, U5 ESP32-S3-WROOM-1

Commit message: finished the PCB, finally
Parts:
- C1, C10, C12, C3, C4: value 10µF -> C15850
- C5, C6: value 1µF -> C28323
- J1: value USB_C_Receptacle_USB2.0_14P -> C165948
- J2: value Micro_SD_Card_Det1 -> C720505; footprint Connector_Card:microSD_HC_Hirose_DM3AT-SF-PEJM5 -> EasyEDA:TF-SMD_TF-115-BCP9
- J3, J4: value Conn_02x04_Odd_Even -> (none)
- J5, J8: value Conn_01x02 -> C160402; footprint Connector_JST:JST_SH_SM02B-SRSS-TB_1x02-1MP_P1.00mm_Horizontal -> EasyEDA:CONN-SMD_2P-P1.00_SM02B-SRSS-TB-LF-SN
- J6, J7: value Conn_01x08 -> C160407; footprint Connector_JST:JST_SH_SM08B-SRSS-TB_1x08-1MP_P1.00mm_Horizontal -> EasyEDA:CONN-TH_SM08B-SRSS-TB-LF-SN
- J9: value Conn_01x02 -> (none)
- Q1: value FS8205A -> C7525054; footprint FS8205A:SOP65P640X120-8N -> EasyEDA:TSSOP-8_L4.4-W3.0-P0.65-LS6.4-BL
- SW4, SW5: value SW_Push -> C139797
- U5: value ESP32-S3-WROOM-1 -> ESP32-S3-WROOM-1-N16-R8
Connections:
- net +3.3V: now also J3.2 (Pin_2); no longer J3.8 (Pin_8), SW5.2
- net GND: now also J3.1 (Pin_1), U1.9 (EPAD); no longer C16.1, C17.1, J2.SH (SHIELD), J3.7 (Pin_7)
- net at J9.1 (Pin_1): now also J8.2 (Pin_2); no longer J8.1 (Pin_1)
- net at J9.2 (Pin_2): now also J8.1 (Pin_1); no longer J8.2 (Pin_2)
- net at U5.17 (IO9): now also J3.5 (Pin_5); no longer J3.3 (Pin_3)
- net at U5.18 (IO10): now also J3.6 (Pin_6); no longer J3.4 (Pin_4)
- net at J7.6 (Pin_6), U5.19 (IO11): now also J3.4 (Pin_4); no longer J3.6 (Pin_6)
- net at J7.5 (Pin_5), U5.20 (IO12): now also J3.3 (Pin_3); no longer J3.5 (Pin_5)
- net at R9.1, U5.3 (EN): now also SW5.2
- net at U5.4 (IO4): now also J3.7 (Pin_7); no longer J3.1 (Pin_1)
- net at U5.5 (IO5): now also J3.8 (Pin_8); no longer J3.2 (Pin_2)
- net at J6.1 (Pin_1): now also J4.8 (Pin_8); no longer J4.1 (Pin_1)
- net at J6.2 (Pin_2): now also J4.7 (Pin_7); no longer J4.2 (Pin_2)
- net at J6.3 (Pin_3): now also J4.6 (Pin_6); no longer J4.3 (Pin_3)
- net at J6.4 (Pin_4): now also J4.5 (Pin_5); no longer J4.4 (Pin_4)
- net at J6.5 (Pin_5): now also J4.4 (Pin_4); no longer J4.5 (Pin_5)
- net at J6.6 (Pin_6): now also J4.3 (Pin_3); no longer J4.6 (Pin_6)
- net at C16.2, C17.2: now also J4.1 (Pin_1), J6.8 (Pin_8); no longer J4.7 (Pin_7), J6.7 (Pin_7)
- new net: C16.1, C17.1, J4.2 (Pin_2), J6.7 (Pin_7)
- no-connect marks 0 -> 1
Other:
- moved on the sheet: R9, SW5

Commit message: fixed jst connector having inverted wiring on the pcb and added nomenclatures for each component
Connections:
- net +3.3V: now also C16.2, C17.2, J4.1 (Pin_1), J6.1 (Pin_1)
- net GND: now also C16.1, C17.1, J4.2 (Pin_2), J6.2 (Pin_2)
- net at J8.2 (Pin_2), J9.1 (Pin_1): now also C2.2, J5.1 (Pin_1), Q1.6, Q1.7, U2.6 (GND)
- net at J8.1 (Pin_1), J9.2 (Pin_2): now also C3.2, C4.1, J5.2 (Pin_2), R7.2, U1.5 (BAT), U3.1 (VIN), U3.3 (EN)
- net at J7.1 (Pin_1), U5.11 (IO18): now also J4.8 (Pin_8), J6.8 (Pin_8)
- net at J7.3 (Pin_3), U5.12 (IO8): now also J4.6 (Pin_6), J6.6 (Pin_6)
- net at J3.4 (Pin_4), J7.6 (Pin_6), U5.19 (IO11): now also J4.3 (Pin_3), J6.3 (Pin_3)
- net at J3.3 (Pin_3), J7.5 (Pin_5), U5.20 (IO12): now also J4.4 (Pin_4), J6.4 (Pin_4)
- net at J7.4 (Pin_4), U5.7 (IO7): now also J4.5 (Pin_5), J6.5 (Pin_5)
- net at J7.2 (Pin_2), U5.8 (IO15): now also J4.7 (Pin_7), J6.7 (Pin_7)
- no-connect marks 1 -> 0
Other:
- moved on the sheet: J6, J8

Commit message: fixed up PCB schematics component values
Parts:
- added C18, C19: 100nF, Capacitor_SMD:C_0805_2012Metric, symbol Device:C_Small
- C1, C10, C12, C3, C4: value C15850 -> 10μF; JLCPCB (none) -> C15850
- C5, C6: value C28323 -> 1μF; JLCPCB (none) -> C28323
- J1: value C165948 -> USB-C-2.0-RECEPTACLE; JLCPCB (none) -> C165948
- J2: value C720505 -> MICRO-SD-CARD-READER; JLCPCB (none) -> C720505
- J5, J8: value C160402 -> JST_SH_01x02_1.0mm; JLCPCB (none) -> C160402
- J6, J7: value C160407 -> JST_SH_02x04_1.0mm; JLCPCB (none) -> C160407
- Q1: value C7525054 -> FS8205A; JLCPCB (none) -> C7525054
- SW4, SW5: value C139797 -> 2_PIN_SW
- U1: JLCPCB (none) -> C139797
Connections:
- net +3.3V: no longer C16.2, C17.2, J4.1 (Pin_1), J6.1 (Pin_1)
- net GND: now also C18.1, C19.1; no longer C16.1, C17.1, J4.2 (Pin_2), J6.2 (Pin_2)
- net at C2.2, J5.1 (Pin_1), Q1.6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: no longer J8.2 (Pin_2), J9.1 (Pin_1)
- net at C3.2, C4.1, J5.2 (Pin_2)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: no longer J8.1 (Pin_1), J9.2 (Pin_2)
- net at R9.1, SW5.2, U5.3 (EN): now also C19.2
- net at J7.1 (Pin_1), U5.11 (IO18): no longer J4.8 (Pin_8), J6.8 (Pin_8)
- net at J7.3 (Pin_3), U5.12 (IO8): no longer J4.6 (Pin_6), J6.6 (Pin_6)
- net at J3.4 (Pin_4), J7.6 (Pin_6), U5.19 (IO11): no longer J4.3 (Pin_3), J6.3 (Pin_3)
- net at J3.3 (Pin_3), J7.5 (Pin_5), U5.20 (IO12): no longer J4.4 (Pin_4), J6.4 (Pin_4)
- net at R15.1, SW4.1, U5.27 (IO0): now also C18.2
- net at J7.4 (Pin_4), U5.7 (IO7): no longer J4.5 (Pin_5), J6.5 (Pin_5)
- net at J7.2 (Pin_2), U5.8 (IO15): no longer J4.7 (Pin_7), J6.7 (Pin_7)
- new net: J8.2 (Pin_2), J9.1 (Pin_1)
- new net: J8.1 (Pin_1), J9.2 (Pin_2)
- new net: C16.2, C17.2, J4.1 (Pin_1), J6.1 (Pin_1)
- new net: C16.1, C17.1, J4.2 (Pin_2), J6.2 (Pin_2)
- new net: J4.3 (Pin_3), J6.3 (Pin_3)
- new net: J4.4 (Pin_4), J6.4 (Pin_4)
- new net: J4.5 (Pin_5), J6.5 (Pin_5)
- new net: J4.6 (Pin_6), J6.6 (Pin_6)
- new net: J4.7 (Pin_7), J6.7 (Pin_7)
- new net: J4.8 (Pin_8), J6.8 (Pin_8)
Other:
- moved on the sheet: R9, SW5

Commit message: made ldo 1uF capacitor a 100uF
Parts:
- C5: value 1μF -> 100μF
Changed lines of the file:
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@@
 		(fields_autoplaced yes)
 		(property "Reference" "C5"
-			(at 331.47 48.2538 0)
+			(at 336.55 45.7135 0)
 			(show_name no)
 			(do_not_autoplace no)
@@
 					(size 1.27 1.27)
 				)
-				(justify left)
+				(justify right)
 			)
 		)
-		(property "Value" "1μF"
-			(at 331.47 45.7138 0)
+		(property "Value" "100μF"
+			(at 336.55 48.2535 0)
 			(show_name no)
 			(do_not_autoplace no)
@@
 					(size 1.27 1.27)
 				)
-				(justify left)
+				(justify right)
 			)
 		)

Commit message: actually swapped the footprint of C5 from 0805 to 1026
Parts:
- C5: footprint Capacitor_SMD:C_0805_2012Metric -> Capacitor_SMD:C_1206_3216Metric
Changed lines of the file:
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@@
 			)
 		)
-		(property "Footprint" "Capacitor_SMD:C_0805_2012Metric"
+		(property "Footprint" "Capacitor_SMD:C_1206_3216Metric"
 			(at 334.01 46.99 0)
 			(hide yes)
